Commit message: removing the fingers so we can use Rethink's joint controller.

File: baxter_description/urdf/baxter_h2r_fingers.urdf (robot description, URDF)
Before this commit: robot baxter, 48 links, 47 joints
Links:
- added link left_gripper_l_finger, mass 0.0001; collision box size=0.01 0.01 0.1; visual mesh filename=package://baxter_description/meshes/electric_gripper/finger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
- added link left_gripper_r_finger, mass 0.00094542; collision box size=0.01 0.01 0.1; visual mesh filename=package://baxter_description/meshes/electric_gripper/finger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
- added link right_gripper_l_finger, mass 0.00094542; collision box size=0.01 0.01 0.1; visual mesh filename=package://baxter_description/meshes/electric_gripper/finger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
- added link right_gripper_r_finger, mass 0.0001; collision box size=0.01 0.01 0.1; visual mesh filename=package://baxter_description/meshes/electric_gripper/finger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
Joints:
- added joint left_gripper_l_finger_joint: type prismatic, parent left_gripper, child left_gripper_l_finger, origin xyz=0.0 0.06 0.035 rpy=0 0 0, axis 0 0 1, limit lower=-0.0125 upper=0.0095 effort=20.0 velocity=5.0
- added joint left_gripper_r_finger_joint: type prismatic, parent left_gripper, child left_gripper_r_finger, origin xyz=0.0 0.06 -0.035 rpy=0 0 0, axis 0 0 1, limit lower=-0.0125 upper=0.0095 effort=20.0 velocity=5.0, mimic joint=left_gripper_l_finger_joint multiplier=-1 offset=0
- added joint right_gripper_l_finger_joint: type prismatic, parent right_gripper, child right_gripper_l_finger, origin xyz=0.0 0.06 0.035 rpy=0 0 0, axis 0 0 1, limit lower=-0.0125 upper=0.0095 effort=20.0 velocity=5.0
- added joint right_gripper_r_finger_joint: type prismatic, parent right_gripper, child right_gripper_r_finger, origin xyz=0.0 0.06 -0.035 rpy=0 0 0, axis 0 0 1, limit lower=-0.0125 upper=0.0095 effort=20.0 velocity=5.0, mimic joint=right_gripper_l_finger_joint multiplier=-1 offset=0
