Commit message: urdf from stephen

File: baxter_description/urdf/baxter.urdf (robot description, URDF)
Before this commit: robot baxter, 54 links, 53 joints
Links:
- removed link display
- removed link left_hand_accelerometer
- link base: mass 0.0001 -> None
- link head: geometry collision sphere radius=0.001; visual mesh filename=package://baxter_description/meshes/head/H0.DAE
- link left_gripper: mass 0.0001 -> 0.00094542; geometry collision cylinder length=0.05 radius=0.0275; visual mesh filename=package://baxter_description/meshes/electric_gripper/electr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
- link left_gripper_l_finger: mass 0.00094542 -> 0.0001; geometry collision box size=0.01 0.01 0.1; visual mesh filename=package://baxter_description/meshes/electric_gripper/finger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
- link left_gripper_r_finger: geometry collision box size=0.01 0.01 0.1; visual mesh filename=package://baxter_description/meshes/electric_gripper/finger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
- link left_hand: geometry collision cylinder length=0.0464 radius=0.04
- link left_hand_range: geometry visual box size=0.005 .02 .005
- link left_lower_elbow: geometry collision cylinder length=0.10 radius=0.06; visual mesh filename=package://baxter_description/meshes/lower_elbow/E1.DAE
- link left_lower_forearm: geometry collision cylinder length=0.10 radius=0.06; visual mesh filename=package://baxter_description/meshes/lower_forearm/W1.DAE
- link left_lower_shoulder: geometry collision cylinder length=0.12 radius=0.06; visual mesh filename=package://baxter_description/meshes/lower_shoulder/S1.DAE
- link left_upper_elbow: geometry collision cylinder length=0.107 radius=0.06; visual mesh filename=package://baxter_description/meshes/upper_elbow/E0.DAE
- link left_upper_forearm: geometry collision cylinder length=0.088 radius=0.06; visual mesh filename=package://baxter_description/meshes/upper_forearm/W0.DAE
- link left_upper_shoulder: geometry collision cylinder length=0.2722 radius=0.06; visual mesh filename=package://baxter_description/meshes/upper_shoulder/S0.DAE
- link left_wrist: geometry collision cylinder length=0.165 radius=0.06; visual mesh filename=package://baxter_description/meshes/wrist/W2.DAE
- link pedestal: mass 60.864 -> 60.86397744; geometry collision box size=0.8 0.8 0.25; collision cylinder length=0.6 radius=0.15
- link right_gripper: mass 0.0001 -> 0.00094542; geometry collision cylinder length=0.05 radius=0.0275; visual mesh filename=package://baxter_description/meshes/electric_gripper/electr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
- link right_gripper_l_finger: geometry collision box size=0.01 0.01 0.1; visual mesh filename=package://baxter_description/meshes/electric_gripper/finger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
- link right_gripper_r_finger: mass 0.00094542 -> 0.0001; geometry collision box size=0.01 0.01 0.1; visual mesh filename=package://baxter_description/meshes/electric_gripper/finger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
- link right_hand: geometry 
- link right_hand_range: geometry visual box size=0.005 .02 .005
- link right_lower_elbow: geometry collision cylinder length=0.10 radius=0.06; visual mesh filename=package://baxter_description/meshes/lower_elbow/E1.DAE
- link right_lower_forearm: geometry collision cylinder length=0.10 radius=0.06; visual mesh filename=package://baxter_description/meshes/lower_forearm/W1.DAE
- link right_lower_shoulder: geometry collision cylinder length=0.12 radius=0.06; visual mesh filename=package://baxter_description/meshes/lower_shoulder/S1.DAE
- link right_upper_elbow: geometry collision cylinder length=0.107 radius=0.06; visual mesh filename=package://baxter_description/meshes/upper_elbow/E0.DAE
- link right_upper_forearm: geometry collision cylinder length=0.088 radius=0.06; visual mesh filename=package://baxter_description/meshes/upper_forearm/W0.DAE
- link right_upper_shoulder: geometry collision cylinder length=0.2722 radius=0.06; visual mesh filename=package://baxter_description/meshes/upper_shoulder/S0.DAE
- link right_wrist: geometry collision cylinder length=0.165 radius=0.06; visual mesh filename=package://baxter_description/meshes/wrist/W2.DAE
- link screen: geometry collision sphere radius=0.001; visual mesh filename=package://baxter_description/meshes/head/H1.DAE
- link torso: mass 35.3365 -> 35.336455; geometry collision mesh filename=package://baxter_description/meshes/torso/base_link_simple.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; visual mesh filename=package://baxter_description/meshes/torso/base_link.DAE
Joints:
- removed joint display_joint
- removed joint left_hand_accelerometer
- joint collision_head_1: axis 0 0 0 -> (none); origin xyz=0.11 0 0.75 rpy=0 -0 0 -> xyz=0.11 0 0.75 rpy=0 0 0
- joint collision_head_2: axis 0 0 0 -> (none); origin xyz=0.11 0 0.75 rpy=0 -0 0 -> xyz=0.11 0 0.75 rpy=0 0 0
- joint dummy: axis 0 0 0 -> (none); origin xyz=0 0 0 rpy=0 -0 0 -> xyz=0 0 0 rpy=0 0 0
- joint head_camera: axis 0 0 0 -> (none); origin xyz=0.12839 0 0.06368 rpy=1.75057 3.87602e-18 1.5708 -> xyz=0.12839 0.0 0.06368 rpy=0.0 0.61073254 0.0
- joint head_nod: axis 0 0 0 -> (none); origin xyz=0.1227 0 0 rpy=1.75057 3.87602e-18 1.5708 -> xyz=.1227 0 0 rpy=1.75057 0 1.57079632679
- joint head_pan: limit lower=-1.5708 upper=1.5708 effort=50000 velocity=10000 -> lower=-1.57079632679 upper=1.57079632679 effort=50000 velocity=10000; origin xyz=0.06 0 0.686 rpy=0 -0 0 -> xyz=0.06 0 0.686 rpy=0 0 0
- joint left_e0: limit lower=-3.05418 upper=3.05418 effort=50 velocity=1.5 -> lower=-3.05417993878 upper=3.05417993878 effort=50.0 velocity=1.5; origin xyz=0.102 0 0 rpy=1.5708 -1.14194e-16    1.5708 -> xyz=0.102 0 0 rpy=1.57079632679 0 1.57079632679
- joint left_e0_fixed: axis 0 0 0 -> 0 0 1; origin xyz=0.107 0 0 rpy=1.5708 -1.14194e-16 1.5708 -> xyz=0.107 0 0 rpy=1.57079632679 0 1.57079632679
- joint left_e1: limit lower=-0.05 upper=2.618 effort=50 velocity=1.5 -> lower=-0.05 upper=2.618 effort=50.0 velocity=1.5; origin xyz=0.069 0 0.26242 rpy=1.57078 -1.57079 -3.14158 -> xyz=0.069 0 0.26242 rpy=-1.57079632679 -1.57079632679 0
- joint left_endpoint: axis 0 0 0 -> (none); origin xyz=0 0 0.045 rpy=0 -0 0 -> xyz=0.0 0 0.025 rpy=0 0 0
- joint left_gripper_base: axis 0 0 0 -> (none); origin xyz=0 0 0 rpy=0 -0 0 -> xyz=0 0 0 rpy=0 0 0
- joint left_hand: axis 0 0 0 -> 0 0 1; origin xyz=0 0 0.11355 rpy=0 -0 0 -> xyz=0 0 0.11355 rpy=0 0 0
- joint left_hand_camera: axis 0 0 0 -> (none); origin xyz=0.03825 0.012 0.015355 rpy=0 0 -1.5708 -> xyz=0.03825 0.012 0.015355 rpy=0 -1.57079633 0
- joint left_hand_camera_axis: axis 0 0 0 -> (none); origin xyz=0.03825    0.012 0 rpy=0 -0 0 -> xyz=0.03825 0.012 0.015355 rpy=0 0 0
- joint left_hand_range: axis 0 0 0 -> (none); origin xyz=0.032    -0.020245 0.0288 rpy=-3.14158 -1.57079 1.57078 -> xyz=0.032 -0.020245 0.0288 rpy=0 -1.57079632679 -1.57079632679
- joint left_s0: limit lower=-1.70168 upper=1.70168 effort=50 velocity=1.5 -> lower=-1.70167993878 upper=1.70167993878 effort=50.0 velocity=1.5; origin xyz=0.055695 0 0.011038 rpy=0 -0 0 -> xyz=0.055695 0 0.011038 rpy=0 0 0
- joint left_s1: limit lower=-2.147 upper=1.047 effort=50 velocity=1.5 -> lower=-2.147 upper=1.047 effort=100.0 velocity=1.5; origin xyz=0.069 0 0.27035 rpy=-1.5708 0 0 -> xyz=0.069 0 0.27035 rpy=-1.57079632679 0 0
- joint left_torso_arm_mount: axis 0 0 0 -> (none); origin xyz=0.0242443 0.220509 0.107602 rpy=-0.00709144    0.0132693 0.790668 -> xyz=0.024645 0.219645 0.118588 rpy=0 0 0.7854
- joint left_torso_itb_fixed: axis 0 0 0 -> (none); origin xyz=-0.08897    0.15593 0.389125 rpy=1.5708 9.26536e-05 -3.14159 -> xyz=-0.08897 0.15593 0.389125 rpy=-1.57079632679 3.1415 0
- joint left_w0: limit lower=-3.059 upper=3.059 effort=15 velocity=4 -> lower=-3.059 upper=3.059 effort=15.0 velocity=4.0; origin xyz=0.10359 0 0 rpy=1.5708 -1.14194e-16 1.5708 -> xyz=0.10359 0 0 rpy=1.57079632679 0 1.57079632679
- joint left_w0_fixed: axis 0 0 0 -> 0 0 1; origin xyz=0.088 0 0 rpy=1.5708 -1.14194e-16 1.5708 -> xyz=0.088 0 0 rpy=1.57079632679 0 1.57079632679
- joint left_w0_to_itb_fixed: axis 0 0 0 -> 0 0 1; origin xyz=-0.0565 0 0.12 rpy=-1.5708 1.14194e-16    1.5708 -> xyz=-0.0565 0 0.12 rpy=-1.57079632679 0 1.57079632679
- joint left_w1: limit lower=-1.5708 upper=2.094 effort=15 velocity=4 -> lower=-1.57079632679 upper=2.094 effort=15.0 velocity=4.0; origin xyz=0.01 0 0.2707 rpy=1.57078    -1.57079 -3.14158 -> xyz=0.01 0 0.2707 rpy=-1.57079632679 -1.57079632679 0
- joint left_w2: limit lower=-3.059 upper=3.059 effort=15 velocity=4 -> lower=-3.059 upper=3.059 effort=15.0 velocity=4.0; origin xyz=0.115975 0 0 rpy=1.5708 -1.14194e-16    1.5708 -> xyz=0.115975 0 0 rpy=1.57079632679 0 1.57079632679
- joint pedestal_fixed: axis 0 0 0 -> (none); origin xyz=0 0 0 rpy=0 -0 0 -> xyz=0.0 0.0 0.0 rpy=0 0 0
- joint right_e0: limit lower=-3.05418 upper=3.05418 effort=50 velocity=1.5 -> lower=-3.05417993878 upper=3.05417993878 effort=50.0 velocity=1.5; origin xyz=0.102 0    0 rpy=1.5708 -1.14194e-16 1.5708 -> xyz=0.102 0 0 rpy=1.57079632679 0 1.57079632679
- joint right_e0_fixed: axis 0 0 0 -> 0 0 1; origin xyz=0.107 0    0 rpy=1.5708 -1.14194e-16 1.5708 -> xyz=0.107 0 0 rpy=1.57079632679 0 1.57079632679
- joint right_e1: limit lower=-0.05 upper=2.618 effort=50 velocity=1.5 -> lower=-0.05 upper=2.618 effort=50.0 velocity=1.5; origin xyz=0.069 0 0.26242 rpy=1.57078 -1.57079 -3.14158 -> xyz=0.069 0 0.26242 rpy=-1.57079632679 -1.57079632679 0
- joint right_endpoint: axis 0 0 0 -> (none); origin xyz=0 0 0.045 rpy=0 -0 0 -> xyz=0.0 0 0.025 rpy=0 0 0
- joint right_gripper_base: axis 0 0 0 -> (none); origin xyz=0 0 0 rpy=0 -0 0 -> xyz=0 0 0 rpy=0 0 0
- joint right_hand: axis 0 0 0 -> 0 0 1; origin xyz=0 0 0.11355 rpy=0 -0 0 -> xyz=0 0 0.11355 rpy=0 0 0
- joint right_hand_accelerometer: axis 0 0 0 -> (none); origin xyz=0.00198 0.000133 -0.0146 rpy=0 -0 0 -> xyz=0.00198 0.000133 -0.0146 rpy=0 0 0
- joint right_hand_camera: axis 0 0 0 -> (none); origin xyz=0.03825 0.012 0.015355 rpy=0 0 -1.5708 -> xyz=0.03825 0.012 0.015355 rpy=0 -1.57079633 0
- joint right_hand_camera_axis: axis 0 0 0 -> (none); origin xyz=0.03825 0.012 0 rpy=0 -0 0 -> xyz=0.03825 0.012 0.015355 rpy=0 0 0
- joint right_hand_range: axis 0 0 0 -> (none); origin xyz=0.032 -0.020245 0.0288 rpy=-3.14158 -1.57079 1.57078 -> xyz=0.032 -0.020245 0.0288 rpy=0 -1.57079632679 -1.57079632679
- joint right_s0: limit lower=-1.70168 upper=1.70168 effort=50 velocity=1.5 -> lower=-1.70167993878 upper=1.70167993878 effort=50.0 velocity=1.5; origin xyz=0.055695 0 0.011038 rpy=0 -0 0 -> xyz=0.055695 0 0.011038 rpy=0 0 0
- joint right_s1: limit lower=-2.147 upper=1.047 effort=50 velocity=1.5 -> lower=-2.147 upper=1.047 effort=100.0 velocity=1.5; origin xyz=0.069 0 0.27035 rpy=-1.5708 0 0 -> xyz=0.069 0 0.27035 rpy=-1.57079632679 0 0
- joint right_torso_arm_mount: axis 0 0 0 -> (none); origin xyz=0.0252076 -0.219127 0.108342 rpy=0.0049102 -0.00625363    -0.785007 -> xyz=0.024645 -0.219645 0.118588 rpy=0 0 -0.7854
- joint right_torso_itb_fixed: axis 0 0 0 -> (none); origin xyz=-0.08897 -0.15593    0.389125 rpy=1.5708 -0 0 -> xyz=-0.08897 -0.15593 0.389125 rpy=1.57079632679 0 0
- joint right_w0: limit lower=-3.059 upper=3.059 effort=15 velocity=4 -> lower=-3.059 upper=3.059 effort=15.0 velocity=4.0; origin xyz=0.10359    0 0 rpy=1.5708 -1.14194e-16 1.5708 -> xyz=0.10359 0 0 rpy=1.57079632679 0 1.57079632679
- joint right_w0_fixed: axis 0 0 0 -> 0 0 1; origin xyz=0.088 0 0 rpy=1.5708 -1.14194e-16 1.5708 -> xyz=0.088 0 0 rpy=1.57079632679 0 1.57079632679
- joint right_w0_to_itb_fixed: axis 0 0 0 -> 0 0 1; origin xyz=-0.0565 0 0.12 rpy=-1.5708 1.14194e-16 1.5708 -> xyz=-0.0565 0 0.12 rpy=-1.57079632679 0 1.57079632679
- joint right_w1: limit lower=-1.5708 upper=2.094 effort=15 velocity=4 -> lower=-1.57079632679 upper=2.094 effort=15.0 velocity=4.0; origin xyz=0.01 0 0.2707 rpy=1.57078 -1.57079    -3.14158 -> xyz=0.01 0 0.2707 rpy=-1.57079632679 -1.57079632679 0
- joint right_w2: limit lower=-3.059 upper=3.059 effort=15 velocity=4 -> lower=-3.059 upper=3.059 effort=15.0 velocity=4.0; origin xyz=0.115975 0 0 rpy=1.5708 -1.14194e-16 1.5708 -> xyz=0.115975 0 0 rpy=1.57079632679 0 1.57079632679
- joint sonar_s0: axis 0 0 0 -> 0 0 1; origin xyz=0.0947 0 0.817 rpy=0 -0 0 -> xyz=0.0947 0 .817 rpy=0 0 0
- joint torso_t0: axis 0 0 0 -> (none); origin xyz=0 0 0 rpy=0 -0 0 -> xyz=0 0 0 rpy=0 0 0
